File: eagle_files/schematic_final.sch (EAGLE design)
At the start: 46 parts, among them IC1 IC_ULN2003-TSSOP-16, T1 BPX81, T2 BPX81, T3 BPX81, T4 BPX81, T5 BPX81, T6 BPX81

Commit message: updated board
Connections:
- removed net DIAG_L_IN: R12.2, T6.E
- removed net DIAG_R_IN: R11.2, T5.E
- removed net FRONT_L_IN: R6.2, T3.E
- removed net FRONT_R_IN: R5.2, T2.E
- removed net SIDE_L_IN: R8.2, T4.E
- removed net SIDE_R_IN: R7.2, T1.E
- net DIAG_L: now also R12.2, T6.E
- net DIAG_R: now also R11.2, T5.E
- net FRONT_L: now also R6.2, T3.E
- net FRONT_R: now also R5.2, T2.E
- net SIDE_L: now also R8.2, T4.E
- net SIDE_R: now also R7.2, T1.E
Other:
- note added: "1.2.0"
- note removed: "1.0.0"
